Commit message: More work on robot_description.

File: sfg_tb4_description/xacro/robot_description.urdf.xacro (robot description, xacro)
@@ -29,3 +29,39 @@
         <origin rpy="${0.5 * pi} 0 ${0.5 * pi}" xyz="0.01774 0 0.092" />
     </xacro:luxonis_oakd_pro>
+    <!-- tracker mount -->
+    <joint name="tracker_mount_joint" type="fixed">
+        <parent link="base" />
+        <child link="tracker_mount" />
+        <origin rpy="0 0 0" xyz="-0.03401 0.08 0.14596" />
+    </joint>
+    <link name="tracker_mount">
+        <visual>
+            <geometry>
+                <mesh filename="package://sfg_tb4_description/mesh/tracker_mount.dae"
+                    scale="1 1 1" />
+            </geometry>
+        </visual>
+    </link>
+    <!-- tracker -->
+    <xacro:htc_vive_tracker_30 name="tracker" parent="tracker_mount">
+        <origin rpy="0 0 ${-0.5 * pi}" xyz="0 0 0.00825" />
+    </xacro:htc_vive_tracker_30>
+    <!-- lidar back mount -->
+    <joint name="lidar_back_mount_joint" type="fixed">
+        <parent link="base" />
+        <child link="lidar_back_mount" />
+        <origin rpy="0 0 0" xyz="-0.03395 -0.08 0.14596" />
+    </joint>
+    <link name="lidar_back_mount">
+        <visual>
+            <geometry>
+                <mesh filename="package://sfg_tb4_description/mesh/lidar_back_mount.dae"
+                    scale="1 1 1" />
+            </geometry>
+        </visual>
+    </link>
+    <!-- lidar back -->
+    <xacro:livox_mid360 name="lidar_back" parent="lidar_back_mount">
+        <origin rpy="0 0 ${-0.5 * pi}" xyz="0.00006 0 0.0065" />
+    </xacro:livox_mid360>
 </robot>

Commit message: Fixed tb4 description still using old sensor names...

File: sfg_tb4_description/xacro/robot_description.urdf.xacro (robot description, xacro)
@@ -11,56 +11,56 @@
         </visual>
     </link>
-    <!-- camera head mount -->
-    <joint name="camera_head_mount_joint" type="fixed">
+    <!-- camera back mount -->
+    <joint name="camera_back_mount_joint" type="fixed">
         <parent link="base" />
-        <child link="camera_head_mount" />
+        <child link="camera_back_mount" />
         <origin rpy="0 0 0" xyz="-0.10001 -0.00001 0.14596" />
     </joint>
-    <link name="camera_head_mount">
+    <link name="camera_back_mount">
         <visual>
             <geometry>
-                <mesh filename="package://sfg_tb4_description/mesh/camera_head_mount.dae"
+                <mesh filename="package://sfg_tb4_description/mesh/camera_back_mount.dae"
                     scale="1 1 1" />
             </geometry>
         </visual>
     </link>
-    <!-- camera head -->
-    <xacro:luxonis_oakd_pro name="camera_head" parent="camera_head_mount">
+    <!-- camera back -->
+    <xacro:luxonis_oakd_pro name="camera_back" parent="camera_back_mount">
         <origin rpy="${0.5 * pi} 0 ${0.5 * pi}" xyz="0.01774 0 0.092" />
     </xacro:luxonis_oakd_pro>
-    <!-- tracker mount -->
-    <joint name="tracker_mount_joint" type="fixed">
+    <!-- tracker left mount -->
+    <joint name="tracker_left_mount_joint" type="fixed">
         <parent link="base" />
-        <child link="tracker_mount" />
+        <child link="tracker_left_mount" />
         <origin rpy="0 0 0" xyz="-0.03401 0.08 0.14596" />
     </joint>
-    <link name="tracker_mount">
+    <link name="tracker_left_mount">
         <visual>
             <geometry>
-                <mesh filename="package://sfg_tb4_description/mesh/tracker_mount.dae"
+                <mesh filename="package://sfg_tb4_description/mesh/tracker_left_mount.dae"
                     scale="1 1 1" />
             </geometry>
         </visual>
     </link>
-    <!-- tracker -->
-    <xacro:htc_vive_tracker_30 name="tracker" parent="tracker_mount">
+    <!-- tracker left -->
+    <xacro:htc_vive_tracker_30 name="tracker_left" parent="tracker_left_mount">
         <origin rpy="0 0 ${-0.5 * pi}" xyz="0 0 0.00825" />
     </xacro:htc_vive_tracker_30>
-    <!-- lidar back mount -->
-    <joint name="lidar_back_mount_joint" type="fixed">
+    <!-- lidar right mount -->
+    <joint name="lidar_right_mount_joint" type="fixed">
         <parent link="base" />
-        <child link="lidar_back_mount" />
+        <child link="lidar_right_mount" />
         <origin rpy="0 0 0" xyz="-0.03395 -0.08 0.14596" />
     </joint>
-    <link name="lidar_back_mount">
+    <link name="lidar_right_mount">
         <visual>
             <geometry>
-                <mesh filename="package://sfg_tb4_description/mesh/lidar_back_mount.dae"
+                <mesh filename="package://sfg_tb4_description/mesh/lidar_right_mount.dae"
                     scale="1 1 1" />
             </geometry>
         </visual>
     </link>
-    <!-- lidar back -->
-    <xacro:livox_mid360 name="lidar_back" parent="lidar_back_mount">
+    <!-- lidar right -->
+    <xacro:livox_mid360 name="lidar_right" parent="lidar_right_mount">
         <origin rpy="0 0 ${-0.5 * pi}" xyz="0.00006 0 0.0065" />
     </xacro:livox_mid360>

Commit message: sfg_tb4_description: Adapted robot_description.urdf.xacro to work with new camera orientation.

File: sfg_tb4_description/xacro/robot_description.urdf.xacro (robot description, xacro)
@@ -27,5 +27,5 @@
     <!-- camera back -->
     <xacro:luxonis_oakd_pro name="camera_back" parent="camera_back_mount">
-        <origin rpy="${0.5 * pi} 0 ${0.5 * pi}" xyz="0.01774 0 0.092" />
+        <origin rpy="${0.5 * pi} ${0.5 * pi} ${0.5 * pi}" xyz="0.01774 0 0.092" />
     </xacro:luxonis_oakd_pro>
     <!-- tracker left mount -->
@@ -63,5 +63,5 @@
     <!-- lidar right -->
     <xacro:livox_mid360 name="lidar_right" parent="lidar_right_mount">
-        <origin rpy="0 0 ${-0.5 * pi}" xyz="0.00006 0 0.0065" />
+        <origin rpy="0 0 ${0.5 * pi}" xyz="0.00006 0 0.0065" />
     </xacro:livox_mid360>
 </robot>

Commit message: Fixed wrong indent size for xacro/xml files.

File: sfg_tb4_description/xacro/robot_description.urdf.xacro (robot description, xacro)
@@ -1,67 +1,67 @@
 <?xml version="1.0"?>
 <robot name="tb4" xmlns:xacro="http://www.ros.org/wiki/xacro">
-    <xacro:include filename="$(find sfg_peripherals_description)/xacro/htc_vive_tracker_30.xacro" />
-    <xacro:include filename="$(find sfg_peripherals_description)/xacro/livox_mid360.xacro" />
-    <xacro:include filename="$(find sfg_peripherals_description)/xacro/luxonis_oakd_pro.xacro" />
-    <link name="base">
-        <visual>
-            <geometry>
-                <mesh filename="package://sfg_tb4_description/mesh/base.dae" scale="1 1 1" />
-            </geometry>
-        </visual>
-    </link>
-    <!-- camera back mount -->
-    <joint name="camera_back_mount_joint" type="fixed">
-        <parent link="base" />
-        <child link="camera_back_mount" />
-        <origin rpy="0 0 0" xyz="-0.10001 -0.00001 0.14596" />
-    </joint>
-    <link name="camera_back_mount">
-        <visual>
-            <geometry>
-                <mesh filename="package://sfg_tb4_description/mesh/camera_back_mount.dae"
-                    scale="1 1 1" />
-            </geometry>
-        </visual>
-    </link>
-    <!-- camera back -->
-    <xacro:luxonis_oakd_pro name="camera_back" parent="camera_back_mount">
-        <origin rpy="${0.5 * pi} ${0.5 * pi} ${0.5 * pi}" xyz="0.01774 0 0.092" />
-    </xacro:luxonis_oakd_pro>
-    <!-- tracker left mount -->
-    <joint name="tracker_left_mount_joint" type="fixed">
-        <parent link="base" />
-        <child link="tracker_left_mount" />
-        <origin rpy="0 0 0" xyz="-0.03401 0.08 0.14596" />
-    </joint>
-    <link name="tracker_left_mount">
-        <visual>
-            <geometry>
-                <mesh filename="package://sfg_tb4_description/mesh/tracker_left_mount.dae"
-                    scale="1 1 1" />
-            </geometry>
-        </visual>
-    </link>
-    <!-- tracker left -->
-    <xacro:htc_vive_tracker_30 name="tracker_left" parent="tracker_left_mount">
-        <origin rpy="0 0 ${-0.5 * pi}" xyz="0 0 0.00825" />
-    </xacro:htc_vive_tracker_30>
-    <!-- lidar right mount -->
-    <joint name="lidar_right_mount_joint" type="fixed">
-        <parent link="base" />
-        <child link="lidar_right_mount" />
-        <origin rpy="0 0 0" xyz="-0.03395 -0.08 0.14596" />
-    </joint>
-    <link name="lidar_right_mount">
-        <visual>
-            <geometry>
-                <mesh filename="package://sfg_tb4_description/mesh/lidar_right_mount.dae"
-                    scale="1 1 1" />
-            </geometry>
-        </visual>
-    </link>
-    <!-- lidar right -->
-    <xacro:livox_mid360 name="lidar_right" parent="lidar_right_mount">
-        <origin rpy="0 0 ${0.5 * pi}" xyz="0.00006 0 0.0065" />
-    </xacro:livox_mid360>
+  <xacro:include filename="$(find sfg_peripherals_description)/xacro/htc_vive_tracker_30.xacro" />
+  <xacro:include filename="$(find sfg_peripherals_description)/xacro/livox_mid360.xacro" />
+  <xacro:include filename="$(find sfg_peripherals_description)/xacro/luxonis_oakd_pro.xacro" />
+  <link name="base">
+    <visual>
+      <geometry>
+        <mesh filename="package://sfg_tb4_description/mesh/base.dae" scale="1 1 1" />
+      </geometry>
+    </visual>
+  </link>
+  <!-- camera back mount -->
+  <joint name="camera_back_mount_joint" type="fixed">
+    <parent link="base" />
+    <child link="camera_back_mount" />
+    <origin rpy="0 0 0" xyz="-0.10001 -0.00001 0.14596" />
+  </joint>
+  <link name="camera_back_mount">
+    <visual>
+      <geometry>
+        <mesh filename="package://sfg_tb4_description/mesh/camera_back_mount.dae"
+          scale="1 1 1" />
+      </geometry>
+    </visual>
+  </link>
+  <!-- camera back -->
+  <xacro:luxonis_oakd_pro name="camera_back" parent="camera_back_mount">
+    <origin rpy="${0.5 * pi} ${0.5 * pi} ${0.5 * pi}" xyz="0.01774 0 0.092" />
+  </xacro:luxonis_oakd_pro>
+  <!-- tracker left mount -->
+  <joint name="tracker_left_mount_joint" type="fixed">
+    <parent link="base" />
+    <child link="tracker_left_mount" />
+    <origin rpy="0 0 0" xyz="-0.03401 0.08 0.14596" />
+  </joint>
+  <link name="tracker_left_mount">
+    <visual>
+      <geometry>
+        <mesh filename="package://sfg_tb4_description/mesh/tracker_left_mount.dae"
+          scale="1 1 1" />
+      </geometry>
+    </visual>
+  </link>
+  <!-- tracker left -->
+  <xacro:htc_vive_tracker_30 name="tracker_left" parent="tracker_left_mount">
+    <origin rpy="0 0 ${-0.5 * pi}" xyz="0 0 0.00825" />
+  </xacro:htc_vive_tracker_30>
+  <!-- lidar right mount -->
+  <joint name="lidar_right_mount_joint" type="fixed">
+    <parent link="base" />
+    <child link="lidar_right_mount" />
+    <origin rpy="0 0 0" xyz="-0.03395 -0.08 0.14596" />
+  </joint>
+  <link name="lidar_right_mount">
+    <visual>
+      <geometry>
+        <mesh filename="package://sfg_tb4_description/mesh/lidar_right_mount.dae"
+          scale="1 1 1" />
+      </geometry>
+    </visual>
+  </link>
+  <!-- lidar right -->
+  <xacro:livox_mid360 name="lidar_right" parent="lidar_right_mount">
+    <origin rpy="0 0 ${0.5 * pi}" xyz="0.00006 0 0.0065" />
+  </xacro:livox_mid360>
 </robot>

Commit message: sfg_tb4_description: Added dedicated wheel links/joints for the robot.

File: sfg_tb4_description/xacro/robot_description.urdf.xacro (robot description, xacro)
@@ -10,4 +10,45 @@
       </geometry>
     </visual>
+  </link>
+  <!-- left wheel -->
+  <joint name="left_wheel_joint" type="continuous">
+    <parent link="base" />
+    <child link="left_wheel" />
+    <origin rpy="${pi/2} 0 0" xyz="-0.0005 0.11755 0.03605" />
+    <axis xyz="0 1 0" />
+  </joint>
+  <link name="left_wheel">
+    <collision>
+      <geometry>
+        <cylinder radius="0.036" length="0.015" />
+      </geometry>
+    </collision>
+  </link>
+  <!-- right wheel -->
+  <joint name="right_wheel_joint" type="continuous">
+    <parent link="base" />
+    <child link="right_wheel" />
+    <origin rpy="${pi/2} 0 0" xyz="-0.0005 -0.11755 0.03605" />
+    <axis xyz="0 1 0" />
+  </joint>
+  <link name="right_wheel">
+    <collision>
+      <geometry>
+        <cylinder radius="0.036" length="0.015" />
+      </geometry>
+    </collision>
+  </link>
+  <!-- caster wheel -->
+  <joint name="caster_wheel_joint" type="fixed">
+    <parent link="base" />
+    <child link="caster_wheel" />
+    <origin rpy="0 0 0" xyz="0.126 0 0.01389" />
+  </joint>
+  <link name="caster_wheel">
+    <collision>
+      <geometry>
+        <sphere radius="0.013" />
+      </geometry>
+    </collision>
   </link>
   <!-- camera back mount -->

Commit message: removed legacy stuff from htc vive tracker

File: sfg_tb4_description/xacro/robot_description.urdf.xacro (robot description, xacro)
@@ -1,5 +1,4 @@
 <?xml version="1.0"?>
 <robot name="tb4" xmlns:xacro="http://www.ros.org/wiki/xacro">
-    <xacro:include filename="$(find sfg_peripherals_description)/xacro/htc_vive_tracker_30.xacro" />
     <xacro:include filename="$(find sfg_peripherals_description)/xacro/livox_mid360.xacro" />
     <xacro:include filename="$(find sfg_peripherals_description)/xacro/luxonis_oakd_pro.xacro" />
@@ -29,22 +28,4 @@
         <origin rpy="${0.5 * pi} ${0.5 * pi} ${0.5 * pi}" xyz="0.01774 0 0.092" />
     </xacro:luxonis_oakd_pro>
-    <!-- tracker left mount -->
-    <joint name="tracker_left_mount_joint" type="fixed">
-        <parent link="base" />
-        <child link="tracker_left_mount" />
-        <origin rpy="0 0 0" xyz="-0.03401 0.08 0.14596" />
-    </joint>
-    <link name="tracker_left_mount">
-        <visual>
-            <geometry>
-                <mesh filename="package://sfg_tb4_description/mesh/tracker_left_mount.dae"
-                    scale="1 1 1" />
-            </geometry>
-        </visual>
-    </link>
-    <!-- tracker left -->
-    <xacro:htc_vive_tracker_30 name="tracker_left" parent="tracker_left_mount">
-        <origin rpy="0 0 ${-0.5 * pi}" xyz="0 0 0.00825" />
-    </xacro:htc_vive_tracker_30>
     <!-- lidar right mount -->
     <joint name="lidar_right_mount_joint" type="fixed">

Commit message: finally fixed

File: sfg_tb4_description/xacro/robot_description.urdf.xacro (robot description, xacro)
@@ -1,94 +1,91 @@
 <?xml version="1.0"?>
 <robot name="tb4" xmlns:xacro="http://www.ros.org/wiki/xacro">
-    <xacro:include filename="$(find sfg_peripherals_description)/xacro/livox_mid360.xacro" />
-    <xacro:include filename="$(find sfg_peripherals_description)/xacro/luxonis_oakd_pro.xacro" />
-    <link name="base">
-        <visual>
-            <geometry>
-                <mesh filename="package://sfg_tb4_description/mesh/base.dae" scale="1 1 1" />
-            </geometry>
-        </visual>
-    </link>
-    <!-- left wheel -->
-    <joint name="left_wheel_joint" type="continuous">
-        <parent link="base" />
-        <child link="left_wheel" />
-        <origin rpy="${pi/2} 0 0" xyz="-0.0005 0.11755 0.03605" />
-        <axis xyz="0 1 0" />
-    </joint>
-    <link name="left_wheel">
-        <collision>
-            <geometry>
-                <cylinder radius="0.036" length="0.015" />
-            </geometry>
-        </collision>
-    </link>
-    <!-- right wheel -->
-    <joint name="right_wheel_joint" type="continuous">
-        <parent link="base" />
-        <child link="right_wheel" />
-        <origin rpy="${pi/2} 0 0" xyz="-0.0005 -0.11755 0.03605" />
-        <axis xyz="0 1 0" />
-    </joint>
-    <link name="right_wheel">
-        <collision>
-            <geometry>
-                <cylinder radius="0.036" length="0.015" />
-            </geometry>
-        </collision>
-    </link>
-    <!-- lidar right mount -->
-    <joint name="lidar_right_mount_joint" type="fixed">
-        <parent link="base" />
-        <child link="lidar_right_mount" />
-        <origin rpy="0 0 0" xyz="-0.03395 -0.08 0.14596" />
-    </joint>
-    <link name="camera_back_mount">
-        <visual>
-            <geometry>
-                <mesh filename="package://sfg_tb4_description/mesh/camera_back_mount.dae"
-                    scale="1 1 1" />
-            </geometry>
-        </visual>
-    </link>
-    <!-- camera back -->
-    <xacro:luxonis_oakd_pro name="camera_back" parent="camera_back_mount">
-        <origin rpy="${0.5 * pi} ${0.5 * pi} ${0.5 * pi}" xyz="0.01774 0 0.092" />
-    </xacro:luxonis_oakd_pro>
-    <!-- tracker left mount -->
-    <joint name="tracker_left_mount_joint" type="fixed">
-        <parent link="base" />
-        <child link="tracker_left_mount" />
-        <origin rpy="0 0 0" xyz="-0.03401 0.08 0.14596" />
-    </joint>
-    <link name="tracker_left_mount">
-        <visual>
-            <geometry>
-                <mesh filename="package://sfg_tb4_description/mesh/tracker_left_mount.dae"
-                    scale="1 1 1" />
-            </geometry>
-        </visual>
-    </link>
-    <!-- tracker left -->
-    <xacro:htc_vive_tracker_30 name="tracker_left" parent="tracker_left_mount">
-        <origin rpy="0 0 ${-0.5 * pi}" xyz="0 0 0.00825" />
-    </xacro:htc_vive_tracker_30>
-    <!-- lidar right mount -->
-    <joint name="lidar_right_mount_joint" type="fixed">
-        <parent link="base" />
-        <child link="lidar_right_mount" />
-        <origin rpy="0 0 0" xyz="-0.03395 -0.08 0.14596" />
-    </joint>
-    <link name="lidar_right_mount">
-        <visual>
-            <geometry>
-                <mesh filename="package://sfg_tb4_description/mesh/lidar_right_mount.dae"
-                    scale="1 1 1" />
-            </geometry>
-        </visual>
-    </link>
-    <!-- lidar right -->
-    <xacro:livox_mid360 name="lidar_right" parent="lidar_right_mount">
-        <origin rpy="0 0 ${0.5 * pi}" xyz="0.00006 0 0.0065" />
-    </xacro:livox_mid360>
+  <xacro:include filename="$(find sfg_peripherals_description)/xacro/livox_mid360.xacro" />
+  <xacro:include filename="$(find sfg_peripherals_description)/xacro/luxonis_oakd_pro.xacro" />
+  <link name="base">
+    <visual>
+      <geometry>
+        <mesh filename="package://sfg_tb4_description/mesh/base.dae" scale="1 1 1" />
+      </geometry>
+    </visual>
+  </link>
+  <!-- left wheel -->
+  <joint name="left_wheel_joint" type="continuous">
+    <parent link="base" />
+    <child link="left_wheel" />
+    <origin rpy="${pi/2} 0 0" xyz="-0.0005 0.11755 0.03605" />
+    <axis xyz="0 1 0" />
+  </joint>
+  <link name="left_wheel">
+    <collision>
+      <geometry>
+        <cylinder radius="0.036" length="0.015" />
+      </geometry>
+    </collision>
+  </link>
+  <!-- right wheel -->
+  <joint name="right_wheel_joint" type="continuous">
+    <parent link="base" />
+    <child link="right_wheel" />
+    <origin rpy="${pi/2} 0 0" xyz="-0.0005 -0.11755 0.03605" />
+    <axis xyz="0 1 0" />
+  </joint>
+  <link name="right_wheel">
+    <collision>
+      <geometry>
+        <cylinder radius="0.036" length="0.015" />
+      </geometry>
+    </collision>
+  </link>
+  <!-- caster wheel -->
+  <joint name="caster_wheel_joint" type="fixed">
+    <parent link="base" />
+    <child link="caster_wheel" />
+    <origin rpy="0 0 0" xyz="0.126 0 0.01389" />
+  </joint>
+  <link name="caster_wheel">
+    <collision>
+      <geometry>
+        <sphere radius="0.013" />
+      </geometry>
+    </collision>
+  </link>
+  <!-- camera back mount -->
+  <joint name="camera_back_mount_joint" type="fixed">
+    <parent link="base" />
+    <child link="camera_back_mount" />
+    <origin rpy="0 0 0" xyz="-0.10001 -0.00001 0.14596" />
+  </joint>
+  <link name="camera_back_mount">
+    <visual>
+      <geometry>
+        <mesh filename="package://sfg_tb4_description/mesh/camera_back_mount.dae"
+          scale="1 1 1" />
+      </geometry>
+    </visual>
+  </link>
+  <!-- camera back -->
+  <xacro:luxonis_oakd_pro name="camera_back" parent="camera_back_mount">
+    <origin rpy="${0.5 * pi} ${0.5 * pi} ${0.5 * pi}" xyz="0.01774 0 0.092" />
+  </xacro:luxonis_oakd_pro>
+  <!-- ToDo tracker left mount -->
+  <!-- ToDo tracker left -->
+  <!-- lidar right mount -->
+  <joint name="lidar_right_mount_joint" type="fixed">
+    <parent link="base" />
+    <child link="lidar_right_mount" />
+    <origin rpy="0 0 0" xyz="-0.03395 -0.08 0.14596" />
+  </joint>
+  <link name="lidar_right_mount">
+    <visual>
+      <geometry>
+        <mesh filename="package://sfg_tb4_description/mesh/lidar_right_mount.dae"
+          scale="1 1 1" />
+      </geometry>
+    </visual>
+  </link>
+  <!-- lidar right -->
+  <xacro:livox_mid360 name="lidar_right" parent="lidar_right_mount">
+    <origin rpy="0 0 ${0.5 * pi}" xyz="0.00006 0 0.0065" />
+  </xacro:livox_mid360>
 </robot>
